File: ncr-pcb/ncr-pcb.kicad_sch (KiCad schematic)
At the start: 2 parts, among them J1 Conn_01x04, U1 Pico

Commit message: added files
Parts:
- added H1, H10, H2, H3, H4, H5, H6, H7, H8, H9: MountingHole, MountingHole:MountingHole_2.7mm_M2.5_DIN965_Pad, symbol Mechanical:MountingHole
- added LED1, LED2, LED3: LED_Small, LED_THT:LED_D3.0mm, symbol Device:LED_Small
- added R1, R2, R3: R_Small, Keebio-Parts:Resistor-Hybrid, symbol Device:R_Small
Connections:
- net GND: now also U1.33 (AGND), LED1.1 (K), LED2.1 (K), LED3.1 (K)
- net COL14: now reaches U1.1 (GPIO0)
- net COL10: now reaches U1.10 (GPIO7)
- net COL9: now reaches U1.11 (GPIO8)
- net COL8: now reaches U1.12 (GPIO9)
- net ROW5: now reaches U1.14 (GPIO10)
- net ROW4: now reaches U1.15 (GPIO11)
- net ROW3: now reaches U1.16 (GPIO12)
- net ROW2: now reaches U1.17 (GPIO13)
- net ROW1: now reaches U1.19 (GPIO14)
- net COL15: now reaches U1.2 (GPIO1)
- net COL7: now reaches U1.20 (GPIO15)
- net ROW0: now reaches U1.21 (GPIO16)
- net COL0: now reaches U1.22 (GPIO17)
- net COL1: now reaches U1.24 (GPIO18)
- net COL2: now reaches U1.25 (GPIO19)
- net COL3: now reaches U1.26 (GPIO20)
- net COL4: now reaches U1.27 (GPIO21)
- net COL5: now reaches U1.29 (GPIO22)
- net COL6: now reaches U1.31 (GPIO26_ADC0)
- net LED2: now reaches U1.32 (GPIO27_ADC1)
- net LED2: now also R2.1
- net LED1: now reaches U1.34 (GPIO28_ADC2)
- net LED1: now also R1.1
- net COL16: now reaches U1.4 (GPIO2)
- net LED3: now reaches U1.5 (GPIO3)
- net LED3: now also R3.1
- net COL13: now reaches U1.6 (GPIO4)
- net COL12: now reaches U1.7 (GPIO5)
- net COL11: now reaches U1.9 (GPIO6)
- new net: LED2.2 (A), R2.2
- new net: LED3.2 (A), R3.2
- new net: LED1.2 (A), R1.2
